Commit message: parameterize camera width/height and fps

File: realsense2_description/gazebo/_d435.gazebo.xacro (robot description, xacro)
@@ -7,105 +7,116 @@
 <robot xmlns:xacro="http://ros.org/wiki/xacro">
   <xacro:macro name="gazebo_d435"
-    params="camera_name reference_link depth_frame color_frame infra1_frame infra2_frame publish_pointcloud:=true">
+    params="camera_name reference_link depth_frame color_frame infra1_frame infra2_frame
+      enable_infra1 enable_infra2 enable_color enable_depth
+      color_width color_height color_fps depth_width depth_height depth_fps
+      publish_pointcloud:=true">
     <!-- Load parameters to model's main link-->
     <xacro:property name="deg_to_rad" value="0.01745329251994329577" />
     <gazebo reference="${reference_link}">
-      <sensor name="${robot_name}_${camera_name}_color" type="camera">
-        <pose relative_to="${color_frame}">0 0 0 0 0 0</pose>
-        <camera name="__default__">
-          <camera_info_topic>${robot_name}/${camera_name}/color/camera_info</camera_info_topic>
-          <horizontal_fov>${69.4*deg_to_rad}</horizontal_fov>
-          <image>
-            <width>1920</width>
-            <height>1080</height>
-            <format>RGB_INT8</format>
-          </image>
-          <clip>
-            <near>0.1</near>
-            <far>100</far>
-          </clip>
-          <noise>
-            <type>gaussian</type>
-            <mean>0.0</mean>
-            <stddev>0.007</stddev>
-          </noise>
-        </camera>
-        <topic>${robot_name}/${camera_name}/color/image_raw</topic>
-        <always_on>1</always_on>
-        <update_rate>30</update_rate>
-        <visualize>1</visualize>
-      </sensor>
-      <sensor name="${robot_name}_${camera_name}_infra1" type="camera">
-        <pose relative_to="${infra1_frame}">0 0 0 0 0 0</pose>
-        <camera name="__default__">
-          <camera_info_topic>${robot_name}/${camera_name}/infra1/camera_info</camera_info_topic>
-          <horizontal_fov>${85.2*deg_to_rad}</horizontal_fov>
-          <image>
-            <width>1280</width>
-            <height>720</height>
-            <format>L_INT8</format>
-          </image>
-          <clip>
-            <near>0.1</near>
-            <far>100</far>
-          </clip>
-          <noise>
-            <type>gaussian</type>
-            <mean>0.0</mean>
-            <stddev>0.05</stddev>
-          </noise>
-        </camera>
-        <topic>${robot_name}/${camera_name}/infra1/image_raw</topic>
-        <always_on>1</always_on>
-        <update_rate>30</update_rate>
-        <visualize>0</visualize>
-      </sensor>
-      <sensor name="${robot_name}_${camera_name}_infra2" type="camera">
-        <pose relative_to="${infra2_frame}">0 0 0 0 0 0</pose>
-        <camera name="__default__">
-          <camera_info_topic>${robot_name}/${camera_name}/infra2/camera_info</camera_info_topic>
-          <horizontal_fov>${85.2*deg_to_rad}</horizontal_fov>
-          <image>
-            <width>1280</width>
-            <height>720</height>
-            <format>L_INT8</format>
-          </image>
-          <clip>
-            <near>0.1</near>
-            <far>100</far>
-          </clip>
-          <noise>
-            <type>gaussian</type>
-            <mean>0.0</mean>
-            <stddev>0.05</stddev>
-          </noise>
-        </camera>
-        <topic>${robot_name}/${camera_name}/infra2/image_raw</topic>
-        <always_on>1</always_on>
-        <update_rate>30</update_rate>
-        <visualize>0</visualize>
-      </sensor>
-      <sensor name="${robot_name}_${camera_name}_depth" type="depth_camera">
-        <pose relative_to="${depth_frame}">0 0 0 0 0 0</pose>
-        <camera name="__default__">
-          <image>
-            <width>1280</width>
-            <height>720</height>
-          </image>
-          <clip>
-            <near>0.1</near>
-            <far>10</far>
-          </clip>
-          <noise>
-            <type>gaussian</type>
-            <mean>0.0</mean>
-            <stddev>0.01</stddev>
-          </noise>
-        </camera>
-        <topic>${robot_name}/${camera_name}/depth/image_rect_raw</topic>
-        <always_on>1</always_on>
-        <update_rate>30</update_rate>
-        <visualize>1</visualize>
-      </sensor>
+      <xacro:if value="${enable_color}">
+        <sensor name="${robot_name}_${camera_name}_color" type="camera">
+          <pose relative_to="${color_frame}">0 0 0 0 0 0</pose>
+          <camera name="__default__">
+            <camera_info_topic>${robot_name}/${camera_name}/color/camera_info</camera_info_topic>
+            <horizontal_fov>${69.4*deg_to_rad}</horizontal_fov>
+            <image>
+              <width>${color_width}</width>
+              <height>${color_height}</height>
+              <format>RGB_INT8</format>
+            </image>
+            <clip>
+              <near>0.1</near>
+              <far>100</far>
+            </clip>
+            <noise>
+              <type>gaussian</type>
+              <mean>0.0</mean>
+              <stddev>0.007</stddev>
+            </noise>
+          </camera>
+          <topic>${robot_name}/${camera_name}/color/image_raw</topic>
+          <always_on>1</always_on>
+          <update_rate>${color_fps}</update_rate>
+          <visualize>0</visualize>
+        </sensor>
+      </xacro:if>
+      <xacro:if value="${enable_infra1}">
+        <sensor name="${robot_name}_${camera_name}_infra1" type="camera">
+          <pose relative_to="${infra1_frame}">0 0 0 0 0 0</pose>
+          <camera name="__default__">
+            <camera_info_topic>${robot_name}/${camera_name}/infra1/camera_info</camera_info_topic>
+            <horizontal_fov>${85.2*deg_to_rad}</horizontal_fov>
+            <image>
+              <width>1280</width>
+              <height>720</height>
+              <format>L_INT8</format>
+            </image>
+            <clip>
+              <near>0.1</near>
+              <far>100</far>
+            </clip>
+            <noise>
+              <type>gaussian</type>
+              <mean>0.0</mean>
+              <stddev>0.05</stddev>
+            </noise>
+          </camera>
+          <topic>${robot_name}/${camera_name}/infra1/image_raw</topic>
+          <always_on>1</always_on>
+          <update_rate>30</update_rate>
+          <visualize>0</visualize>
+        </sensor>
+      </xacro:if>
+      <xacro:if value="${enable_infra2}">
+        <sensor name="${robot_name}_${camera_name}_infra2" type="camera">
+          <pose relative_to="${infra2_frame}">0 0 0 0 0 0</pose>
+          <camera name="__default__">
+            <camera_info_topic>${robot_name}/${camera_name}/infra2/camera_info</camera_info_topic>
+            <horizontal_fov>${85.2*deg_to_rad}</horizontal_fov>
+            <image>
+              <width>1280</width>
+              <height>720</height>
+              <format>L_INT8</format>
+            </image>
+            <clip>
+              <near>0.1</near>
+              <far>100</far>
+            </clip>
+            <noise>
+              <type>gaussian</type>
+              <mean>0.0</mean>
+              <stddev>0.05</stddev>
+            </noise>
+          </camera>
+          <topic>${robot_name}/${camera_name}/infra2/image_raw</topic>
+          <always_on>1</always_on>
+          <update_rate>30</update_rate>
+          <visualize>0</visualize>
+        </sensor>
+      </xacro:if>
+      <xacro:if value="${enable_depth}">
+        <sensor name="${robot_name}_${camera_name}_depth" type="depth_camera">
+          <pose relative_to="${depth_frame}">0 0 0 0 0 0</pose>
+          <camera name="__default__">
+            <image>
+              <width>${depth_width}</width>
+              <height>${depth_height}</height>
+            </image>
+            <clip>
+              <near>0.1</near>
+              <far>10</far>
+            </clip>
+            <noise>
+              <type>gaussian</type>
+              <mean>0.0</mean>
+              <stddev>0.01</stddev>
+            </noise>
+          </camera>
+          <topic>${robot_name}/${camera_name}/depth/image_rect_raw</topic>
+          <always_on>1</always_on>
+          <update_rate>${depth_fps}</update_rate>
+          <visualize>0</visualize>
+        </sensor>
+      </xacro:if>
     </gazebo>
   </xacro:macro>

File: realsense2_description/urdf/_d435.urdf.xacro (robot description, xacro)
@@ -24,5 +24,7 @@
   <xacro:include filename="$(find realsense2_description)/urdf/_materials.urdf.xacro" />
   <xacro:include filename="$(find realsense2_description)/urdf/_usb_plug.urdf.xacro" />
-  <xacro:macro name="sensor_d435" params="parent *origin name:=camera use_nominal_extrinsics:=false add_plug:=false use_mesh:=true gazebo:=false">
+  <xacro:macro name="sensor_d435" params="parent *origin name:=camera use_nominal_extrinsics:=false add_plug:=false use_mesh:=true gazebo:=false
+    enable_infra1:=false enable_infra2:=false enable_color:=true enable_depth:=true
+    color_width:=1920 color_height:=1080 color_fps:=30 depth_width:=1280 depth_height:=720 depth_fps:=30">
     <xacro:property name="M_PI" value="3.1415926535897931" />
     <!-- The following values are approximate, and the camera node
@@ -158,4 +160,7 @@
         infra1_frame="${name}_infra1_frame"
         infra2_frame="${name}_infra2_frame"
+        enable_infra1="${enable_infra1}" enable_infra2="${enable_infra2}" enable_color="${enable_color}" enable_depth="${enable_depth}"
+        color_width="${color_width}" color_height="${color_height}" color_fps="${color_fps}"
+        depth_width="${depth_width}" depth_height="${depth_height}" depth_fps="${depth_fps}"
         publish_pointcloud="true" />
     </xacro:if>

Commit message: add robot name to description

File: realsense2_description/gazebo/_d435.gazebo.xacro (robot description, xacro)
@@ -7,5 +7,5 @@
 <robot xmlns:xacro="http://ros.org/wiki/xacro">
   <xacro:macro name="gazebo_d435"
-    params="camera_name reference_link depth_frame color_frame infra1_frame infra2_frame
+    params="robot_name camera_name reference_link depth_frame color_frame infra1_frame infra2_frame
       enable_infra1 enable_infra2 enable_color enable_depth
       color_width color_height color_fps depth_width depth_height depth_fps
@@ -97,5 +97,5 @@
       <xacro:if value="${enable_depth}">
         <sensor name="${robot_name}_${camera_name}_depth" type="depth_camera">
-          <pose relative_to="${depth_frame}">0 0 0 0 0 0</pose>
+          <pose relative_to="${color_frame}">0 0 0 0 0 0</pose>
           <camera name="__default__">
             <image>
@@ -105,5 +105,5 @@
             <clip>
               <near>0.1</near>
-              <far>10</far>
+              <far>100</far>
             </clip>
             <noise>

File: realsense2_description/urdf/_d435.urdf.xacro (robot description, xacro)
@@ -24,5 +24,5 @@
   <xacro:include filename="$(find realsense2_description)/urdf/_materials.urdf.xacro" />
   <xacro:include filename="$(find realsense2_description)/urdf/_usb_plug.urdf.xacro" />
-  <xacro:macro name="sensor_d435" params="parent *origin name:=camera use_nominal_extrinsics:=false add_plug:=false use_mesh:=true gazebo:=false
+  <xacro:macro name="sensor_d435" params="parent *origin robot_name:=robot name:=camera use_nominal_extrinsics:=false add_plug:=false use_mesh:=true gazebo:=false
     enable_infra1:=false enable_infra2:=false enable_color:=true enable_depth:=true
     color_width:=1920 color_height:=1080 color_fps:=30 depth_width:=1280 depth_height:=720 depth_fps:=30">
@@ -155,5 +155,6 @@
     <!-- Add Gazebo Sim sensors -->
     <xacro:if value="${gazebo}">
-      <xacro:gazebo_d435 camera_name="${name}" reference_link="${name}_link"
+      <xacro:gazebo_d435 robot_name="${robot_name}"
+        camera_name="${name}" reference_link="${name}_link"
         depth_frame="${name}_depth_frame"
         color_frame="${name}_color_frame"
